File: dc_dc_ext.kicad_sch (KiCad schematic)
At the start: 30 parts, among them U10 TPS56339DDC, U11 TPS56339DDC

Commit message: more 'LCSC' fields in sch files changed to 'LCSC Part'
Parts:
- C47, C53, C54, C60: LCSC C49678 -> (none); LCSC Part (none) -> C49678
- C48, C49, C55, C56: LCSC C49217 -> (none); LCSC Part (none) -> C49217
- C50, C57: LCSC C403725 -> (none); LCSC Part (none) -> C403725
- C51, C52, C58, C59: LCSC C13585 -> (none); LCSC Part (none) -> C13585
- F1, F2: LCSC C883136 -> (none); LCSC Part (none) -> C883136
- L2: LCSC C167220 -> (none); LCSC Part (none) -> C167220
- L3: LCSC C386869 -> (none); LCSC Part (none) -> C386869
- R42: LCSC C22765 -> (none); LCSC Part (none) -> C22765
- R43: LCSC C22984 -> (none); LCSC Part (none) -> C22984
- R44, R48: LCSC C23140 -> (none); LCSC Part (none) -> C23140
- R45, R49: LCSC C25804 -> (none); LCSC Part (none) -> C25804
- R46: LCSC C22940 -> (none); LCSC Part (none) -> C22940
- R47: LCSC C23196 -> (none); LCSC Part (none) -> C23196
- U10, U11: LCSC C2071106 -> (none); LCSC Part (none) -> C2071106
Changed lines of the file:
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@@
     (property "Hold" "Hold: 3A" (id 4) (at 205.74 107.95 90))
     (property "Trip" "Trip: 6A" (id 5) (at 205.74 110.49 90))
-    (property "LCSC" "C883136" (id 6) (at 205.74 105.41 0)
+    (property "LCSC Part" "C883136" (id 6) (at 205.74 105.41 0)
       (effects (font (size 1.27 1.27)) hide)
     )
@@
       (effects (font (size 1.27 1.27)) hide)
     )
-    (property "LCSC" "C386869" (id 5) (at 167.64 118.745 0)
+    (property "LCSC Part" "C386869" (id 5) (at 167.64 118.745 0)
       (effects (font (size 1.27 1.27)) hide)
     )
@@
       (effects (font (size 1.27 1.27)) hide)
     )
-    (property "LCSC" "C22765" (id 4) (at 173.99 42.545 0)
+    (property "LCSC Part" "C22765" (id 4) (at 173.99 42.545 0)
       (effects (font (size 1.27 1.27)) hide)
     )
@@
       (effects (font (size 1.27 1.27)) hide)
     )
-    (property "LCSC" "C49217" (id 4) (at 185.42 52.705 0)
+    (property "LCSC Part" "C49217" (id 4) (at 185.42 52.705 0)
       (effects (font (size 1.27 1.27)) hide)
     )
@@
       (effects (font (size 1.27 1.27)) hide)
     )
-    (property "LCSC" "C2071106" (id 4) (at 137.16 118.745 0)
+    (property "LCSC Part" "C2071106" (id 4) (at 137.16 118.745 0)
       (effects (font (size 1.27 1.27)) hide)
     )
@@
       (effects (font (size 1.27 1.27)) hide)
     )
-    (property "LCSC" "C49678" (id 4) (at 106.68 121.285 0)
+    (property "LCSC Part" "C49678" (id 4) (at 106.68 121.285 0)
       (effects (font (size 1.27 1.27)) hide)
     )
@@
       (effects (font (size 1.27 1.27)) hide)
     )
-    (property "LCSC" "C25804" (id 4) (at 173.99 128.905 0)
+    (property "LCSC Part" "C25804" (id 4) (at 173.99 128.905 0)
       (effects (font (size 1.27 1.27)) hide)
     )
@@
       (effects (font (size 1.27 1.27)) hide)
     )
-    (property "LCSC" "C403725" (id 5) (at 71.12 121.285 0)
+    (property "LCSC Part" "C403725" (id 5) (at 71.12 121.285 0)
       (effects (font (size 1.27 1.27)) hide)
     )
@@
       (effects (font (size 1.27 1.27)) hide)
     )
-    (property "LCSC" "C13585" (id 4) (at 95.25 53.975 0)
+    (property "LCSC Part" "C13585" (id 4) (at 95.25 53.975 0)
       (effects (font (size 1.27 1.27)) hide)
     )
@@
       (effects (font (size 1.27 1.27)) hide)
     )
-    (property "LCSC" "C23196" (id 4) (at 173.99 117.475 0)
+    (property "LCSC Part" "C23196" (id 4) (at 173.99 117.475 0)
       (effects (font (size 1.27 1.27)) hide)
     )
@@
       (effects (font (size 1.27 1.27)) hide)
     )
-    (property "LCSC" "C49217" (id 4) (at 196.85 52.705 0)
+    (property "LCSC Part" "C49217" (id 4) (at 196.85 52.705 0)
       (effects (font (size 1.27 1.27)) hide)
     )
@@
       (effects (font (size 1.27 1.27)) hide)
     )
-    (property "LCSC" "C23140" (id 4) (at 151.13 51.435 0)
+    (property "LCSC Part" "C23140" (id 4) (at 151.13 51.435 0)
       (effects (font (size 1.27 1.27)) hide)
     )
@@
       (effects (font (size 1.27 1.27)) hide)
     )
-    (property "LCSC" "C2071106" (id 4) (at 137.16 51.435 0)
+    (property "LCSC Part" "C2071106" (id 4) (at 137.16 51.435 0)
       (effects (font (size 1.27 1.27)) hide)
     )
@@
       (effects (font (size 1.27 1.27)) hide)
     )
-    (property "LCSC" "C49678" (id 4) (at 158.75 51.435 0)
+    (property "LCSC Part" "C49678" (id 4) (at 158.75 51.435 0)
       (effects (font (size 1.27 1.27)) hide)
     )
@@
       (effects (font (size 1.27 1.27)) hide)
     )
-    (property "LCSC" "C23140" (id 4) (at 151.13 118.745 0)
+    (property "LCSC Part" "C23140" (id 4) (at 151.13 118.745 0)
       (effects (font (size 1.27 1.27)) hide)
     )
@@
       (effects (font (size 1.27 1.27)) hide)
     )
-    (property "LCSC" "C22984" (id 4) (at 173.99 50.165 0)
+    (property "LCSC Part" "C22984" (id 4) (at 173.99 50.165 0)
       (effects (font (size 1.27 1.27)) hide)
     )
@@
     (property "Hold" "Hold: 3A" (id 4) (at 205.74 40.64 90))
     (property "Trip" "Trip: 6A" (id 5) (at 205.74 43.18 90))
-    (property "LCSC" "C883136" (id 6) (at 205.74 38.1 0)
+    (property "LCSC Part" "C883136" (id 6) (at 205.74 38.1 0)
       (effects (font (size 1.27 1.27)) hide)
     )
@@
       (effects (font (size 1.27 1.27)) hide)
     )
-    (property "LCSC" "C13585" (id 4) (at 83.82 121.285 0)
+    (property "LCSC Part" "C13585" (id 4) (at 83.82 121.285 0)
       (effects (font (size 1.27 1.27)) hide)
     )
@@
       (effects (font (size 1.27 1.27)) hide)
     )
-    (property "LCSC" "C25804" (id 4) (at 173.99 61.595 0)
+    (property "LCSC Part" "C25804" (id 4) (at 173.99 61.595 0)
       (effects (font (size 1.27 1.27)) hide)
     )
@@
       (effects (font (size 1.27 1.27)) hide)
     )
-    (property "LCSC" "C22940" (id 4) (at 173.99 109.855 0)
+    (property "LCSC Part" "C22940" (id 4) (at 173.99 109.855 0)
       (effects (font (size 1.27 1.27)) hide)
     )
@@
       (effects (font (size 1.27 1.27)) hide)
     )
-    (property "LCSC" "C49678" (id 4) (at 158.75 118.745 0)
+    (property "LCSC Part" "C49678" (id 4) (at 158.75 118.745 0)
       (effects (font (size 1.27 1.27)) hide)
     )
@@
       (effects (font (size 1.27 1.27)) hide)
     )
-    (property "LCSC" "C49217" (id 4) (at 196.85 120.015 0)
+    (property "LCSC Part" "C49217" (id 4) (at 196.85 120.015 0)
       (effects (font (size 1.27 1.27)) hide)
     )
@@
       (effects (font (size 1.27 1.27)) hide)
     )
-    (property "LCSC" "C167220" (id 5) (at 167.64 51.435 0)
+    (property "LCSC Part" "C167220" (id 5) (at 167.64 51.435 0)
       (effects (font (size 1.27 1.27)) hide)
     )
@@
       (effects (font (size 1.27 1.27)) hide)
     )
-    (property "LCSC" "C49217" (id 4) (at 185.42 120.015 0)
+    (property "LCSC Part" "C49217" (id 4) (at 185.42 120.015 0)
       (effects (font (size 1.27 1.27)) hide)
     )
@@
       (effects (font (size 1.27 1.27)) hide)
     )
-    (property "LCSC" "C13585" (id 4) (at 95.25 121.285 0)
+    (property "LCSC Part" "C13585" (id 4) (at 95.25 121.285 0)
       (effects (font (size 1.27 1.27)) hide)
     )
@@
       (effects (font (size 1.27 1.27)) hide)
     )
-    (property "LCSC" "C403725" (id 5) (at 71.12 53.975 0)
+    (property "LCSC Part" "C403725" (id 5) (at 71.12 53.975 0)
       (effects (font (size 1.27 1.27)) hide)
     )
@@
       (effects (font (size 1.27 1.27)) hide)
     )
-    (property "LCSC" "C49678" (id 4) (at 106.68 53.975 0)
+    (property "LCSC Part" "C49678" (id 4) (at 106.68 53.975 0)
       (effects (font (size 1.27 1.27)) hide)
     )
@@
       (effects (font (size 1.27 1.27)) hide)
     )
-    (property "LCSC" "C13585" (id 4) (at 83.82 53.975 0)
-      (effects (font (size 1.27 1.27)) hide)
-    )
+    (property "LCSC Part" "C13585" (id 4) (at 83.82 53.975 0)
+      (effects (font (size 1.27 1.27)) hide)
+    )

Commit message: corrected LCSC for 4.7uH inductors
Parts:
- L2: LCSC Part C167220 -> C167230
Changed lines of the file:
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@@
       (effects (font (size 1.27 1.27)) hide)
     )
-    (property "Datasheet" "https://datasheet.lcsc.com/lcsc/1811132109_cjiang-Changjiang-Microelectronics-Tech-FXL0630-4R7-M_C167220.pdf" (id 3) (at 167.64 51.435 0)
+    (property "Datasheet" "https://datasheet.lcsc.com/lcsc/1806150431_cjiang--Changjiang-Microelectronics-Tech-FXL1040-4R7-M_C167230.pdf" (id 3) (at 167.64 51.435 0)
       (effects (font (size 1.27 1.27)) hide)
     )
@@
       (effects (font (size 1.27 1.27)) hide)
     )
-    (property "LCSC Part" "C167220" (id 5) (at 167.64 51.435 0)
+    (property "LCSC Part" "C167230" (id 5) (at 167.64 51.435 0)
       (effects (font (size 1.27 1.27)) hide)
     )

Commit message: corrected LCSC of 22uF caps
Parts:
- C48, C49, C55, C56: LCSC Part C49217 -> C12891
Changed lines of the file:
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@@
       (effects (font (size 1.27 1.27)) hide)
     )
-    (property "LCSC Part" "C49217" (id 4) (at 185.42 52.705 0)
+    (property "LCSC Part" "C12891" (id 4) (at 185.42 52.705 0)
       (effects (font (size 1.27 1.27)) hide)
     )
@@
       (effects (font (size 1.27 1.27)) hide)
     )
-    (property "LCSC Part" "C49217" (id 4) (at 196.85 52.705 0)
+    (property "LCSC Part" "C12891" (id 4) (at 196.85 52.705 0)
       (effects (font (size 1.27 1.27)) hide)
     )
@@
       (effects (font (size 1.27 1.27)) hide)
     )
-    (property "LCSC Part" "C49217" (id 4) (at 196.85 120.015 0)
+    (property "LCSC Part" "C12891" (id 4) (at 196.85 120.015 0)
       (effects (font (size 1.27 1.27)) hide)
     )
@@
       (effects (font (size 1.27 1.27)) hide)
     )
-    (property "LCSC Part" "C49217" (id 4) (at 185.42 120.015 0)
-      (effects (font (size 1.27 1.27)) hide)
-    )
+    (property "LCSC Part" "C12891" (id 4) (at 185.42 120.015 0)
+      (effects (font (size 1.27 1.27)) hide)
+    )
